File: MIKOTO RIG.kicad_pcb (KiCad board)
At the start: 2 copper layers, 30 parts, among them J1 Conn_01x05_Female, J2 Conn_01x05_Female, J3 Conn_01x04_Male, J4 Conn_01x04_Male, J5 Conn_01x04_Male, J6 USB_B_Micro, SW1 SW_SPDT, U1 AMS1117-3.3, U2 STM32F405RGT6, Y1 16MHz

Commit message: updated schematics
Done adding sensors, next is to add power inlet and then start on routing
Parts:
- removed J4: Conn_01x04_Male, Connector_PinHeader_2.54mm:PinHeader_1x04_P2.54mm_Vertical
- added C14: 100n, Capacitor_SMD:C_0805_2012Metric, F.Cu at (165.1, 68.6)
- added C15: 100n, Capacitor_SMD:C_0805_2012Metric, F.Cu at (157.6, 77.6)
- added C16: 100n, Capacitor_SMD:C_0805_2012Metric, F.Cu at (152.5, 79.9)
- added C17: 100n, Capacitor_SMD:C_0805_2012Metric, F.Cu at (157.6, 74.6)
- added C18: 100n, Capacitor_SMD:C_0805_2012Metric, F.Cu at (160.7, 71.6)
- added C19: 100n, Capacitor_SMD:C_0805_2012Metric, F.Cu at (160.7, 68.6)
- added IC1: W25N01GVZEIG, SamacSys_Parts:SON127P800X600X80-9N-D, F.Cu at (148.6, 70.9)
- added IC2: BMM150, SamacSys_Parts:BMM150, F.Cu at (156.1, 70.0)
- added IC3: BMI088, SamacSys_Parts:BMI088, F.Cu at (146.9, 78.1)
- added IC4: bmp280, SamacSys_Parts:8-PIN-METAL-LID-LGA, F.Cu at (168.9, 68.9)
- added LED1: 19-237_R6GHBHC-A01_2T, SamacSys_Parts:19237R6GHBHCA012T, F.Cu at (153.1, 76.6)
- added R6: 47, Resistor_SMD:R_0805_2012Metric, F.Cu at (165.1, 71.6)
- added R7: R, Resistor_SMD:R_0805_2012Metric, F.Cu at (162.0, 74.6)
- added R8: R, Resistor_SMD:R_0805_2012Metric, F.Cu at (162.0, 77.5)
- added R9: R, Resistor_SMD:R_0805_2012Metric, F.Cu at (156.9, 80.6)
- C13: value 1u -> 100n
- J1: value Conn_01x05_Female -> Conn_02x05_Odd_Even; footprint Connector_PinHeader_2.54mm:PinHeader_1x05_P2.54mm_Vertical -> Connector_PinSocket_1.27mm:PinSocket_2x05_P1.27mm_Vertical_SMD
- J2: value Conn_01x05_Female -> Conn_01x04_Male; footprint Connector_PinHeader_2.54mm:PinHeader_1x05_P2.54mm_Vertical -> Connector_PinHeader_2.54mm:PinHeader_1x04_P2.54mm_Vertical
- J3: value Conn_01x04_Male -> Conn_01x06_Male; footprint Connector_PinHeader_2.54mm:PinHeader_1x04_P2.54mm_Vertical -> Connector_PinHeader_2.54mm:PinHeader_1x06_P2.54mm_Vertical
- R3, R4: value 1k5 -> 10K
Connections:
- C4 pad 1: /NRST -> +3V3
- C8 pad 1: /RCC_OSC_OUT -> Net-(C8-Pad1)
- FB1 pad 1: +3.3VA -> +3V3
- FB1 pad 2: +3V3 -> +3.3VA
- J1 pad 2: /SPI3_MOSI -> SYS_JTMS-SWDIO
- J1 pad 3: /SPI3_MISO -> GND
- J1 pad 4: /SPI3_SCK -> SYS_JTCK-SWCLK
- J2 pad 2: /SPI1_SCK -> UART4_TX
- J2 pad 3: /SPI1_MISO -> UART4_RX
- J2 pad 4: /SPI1_MOSI -> GND
- J3 pad 1: +3V3 -> GND
- J3 pad 2: /SYS_JTMS-SWDIO -> SPI3_!CS
- J3 pad 3: /SYS_JTCK-SWCLK -> SPI3_MOSI
- J3 pad 4: GND -> SPI3_MISO
- R3 pad 1: /I2C1_SDA -> FLASH!WP
- R4 pad 1: /I2C1_SDA -> +3V3
- R4 pad 2: +3V3 -> FLASH_!HOLD
- U2 pad 14: /UART4_TX -> UART4_TX
- U2 pad 15: /UART4_RX -> TIM2_CH2
- U2 pad 16: unconnected-(U2-Pad16) -> TIM2_CH3
- U2 pad 17: unconnected-(U2-Pad17) -> TIM2_CH4
- U2 pad 20: unconnected-(U2-Pad20) -> SPI1_!NCS_ACC
- U2 pad 21: /SPI1_SCK -> SPI1_SCK
- U2 pad 22: /SPI1_MISO -> SPI1_MISO
- U2 pad 23: /SPI1_MOSI -> SPI1_MOSI
- U2 pad 24: unconnected-(U2-Pad24) -> SPI1_!NCS_GYRO
- U2 pad 25: unconnected-(U2-Pad25) -> INT_ACC
- U2 pad 26: unconnected-(U2-Pad26) -> INT_GYRO
- U2 pad 27: unconnected-(U2-Pad27) -> SPI1_!CS_MAG
- U2 pad 28: unconnected-(U2-Pad28) -> INT_MAG
- U2 pad 29: unconnected-(U2-Pad29) -> SPI1_!CS_BARO
- U2 pad 37: unconnected-(U2-Pad37) -> FLASH!WP
- U2 pad 38: unconnected-(U2-Pad38) -> FLASH_!HOLD
- U2 pad 41: unconnected-(U2-Pad41) -> SPI1_!CS_FLASH
- U2 pad 46: /SYS_JTMS-SWDIO -> SYS_JTMS-SWDIO
- U2 pad 49: /SYS_JTCK-SWCLK -> SYS_JTCK-SWCLK
- U2 pad 51: /SPI3_SCK -> SPI3_SCK
- U2 pad 52: /SPI3_MISO -> UART4_RX
- U2 pad 53: /SPI3_MOSI -> SPI3_MOSI
- U2 pad 54: unconnected-(U2-Pad54) -> SPI3_!CS
- U2 pad 55: unconnected-(U2-Pad55) -> SYS_JTDO_SWO
- U2 pad 56: unconnected-(U2-Pad56) -> SPI3_MISO
- U2 pad 59: /I2C1_SDA -> unconnected-(U2-Pad59)
- U2 pad 61: /I2C1_SCL -> unconnected-(U2-Pad61)
- U2 pad 7: /NRST -> NRST
- Y1 pad 3: /RCC_OSC_OUT -> Net-(C8-Pad1)
